File: bosch_kf3_diodematrix.sch (KiCad schematic (older format))
At the start: 49 parts, among them J1 GS3, J10 GS3, J11 GS3, J12 GS3, J13 GS3, J14 GS3, J15 GS3, J16 GS3, J17 GS2, J18 GS2, J19 GS2, J2 GS3, J20 GS2, J21 GS2, J22 GS2, J23 GS2, J24 GS2, J25 GS2, J26 GS2, J27 GS2, J28 GS2, J29 GS2, J3 GS3, J30 GS2, J31 GS2, J32 GS2, J4 GS3, J5 GS3, J6 GS3, J7 GS3, J8 GS3, J9 GS3, U1 PLL

Commit message: Updated project to KiCad 5
Parts:
- D1, D10, D11, D12, D13, D14, D15, D16, D2, D3, D4, D5, D6, D7, D8, D9: symbol D -> Device:D
- J1, J10, J11, J12, J13, J14, J15, J16, J2, J3, J4, J5, J6, J7, J8, J9: symbol GS3 -> bosch_kf3_diodematrix-rescue:GS3
- J17, J18, J19, J20, J21, J22, J23, J24, J25, J26, J27, J28, J29, J30, J31, J32: symbol GS2 -> bosch_kf3_diodematrix-rescue:GS2
- U1: symbol PLL -> bosch_kf3_diodematrix-rescue:PLL
